File: lisn.kicad_pcb (KiCad board)
At the start: 2 copper layers, 94.2 x 57.4 mm, 68 parts, among them X1 SMA, X13 Contact, X14 Contact, X15 Contact, X16 Contact, X2 Conn_01x01, X4 691313710002, X8 Coax

Commit message: finalize cleanup
Parts:
- removed RR6: 6, Resistor_SMD:R_0603_1608Metric
- added R50: 470kR, Resistor_SMD:R_0603_1608Metric, B.Cu at (113.3, 92.2)
- added R51: 470kR, Resistor_SMD:R_0603_1608Metric, B.Cu at (113.3, 107.8)
- added R6: 27R, Resistor_SMD:R_0603_1608Metric, B.Cu at (139.2, 94.8)
- added X10: Coax, Jumper_Coax:Jumper_RG178, B.Cu at (125.5, 94.8)
- added X11: Coax, Jumper_Coax:Jumper_RG178, B.Cu at (109.2, 80.8)
- added X12: Coax, Jumper_Coax:Jumper_RG178, B.Cu at (125.5, 105.2)
- added X3: 23.3000-22, Connector_STAUBLI:STAUBLI_23.3000-22_Red, F.Cu at (166.8, 84.0)
- added X5: 23.3000-21, Connector_STAUBLI:STAUBLI_23.3000-21_Black, F.Cu at (100.0, 116.0)
- added X6: 23.3000-21, Connector_STAUBLI:STAUBLI_23.3000-21_Black, F.Cu at (166.8, 116.0)
- added X7: 23.3000-24, Connector_STAUBLI:STAUBLI_23.3000-24_Yellow, F.Cu at (100.0, 100.0)
- added X9: Coax, Jumper_Coax:Jumper_RG178, B.Cu at (125.6, 74.8)
- X13, X14, X15, X16: footprint TestPoint:TestPoint_Keystone_5019_Miniature -> SpringContact_Wurth:Wurth_331161702513
- X2: value Conn_01x01 -> 23.3000-22; footprint Connector:Banana_Jack_1Pin -> Connector_STAUBLI:STAUBLI_23.3000-22_Red
- X8: value Coax -> SMA
- moved D11 151.5 mm to (130.7, 78.2)
- moved C1 151.4 mm to (143.6, 94.8)
- moved C10 151.4 mm to (103.0, 107.8)
- moved C12 151.4 mm to (161.1, 106.7)
- moved C13 151.4 mm to (143.6, 105.2)
- moved C14 151.4 mm to (152.6, 105.2)
- moved C2 151.4 mm to (152.6, 94.8)
- moved C3 151.4 mm to (161.1, 93.3)
- moved C5 151.4 mm to (109.6, 92.2)
- moved C6 151.4 mm to (99.5, 92.2)
- moved C7 151.4 mm to (103.0, 92.2)
- moved C8 151.4 mm to (109.6, 107.8)
- moved C9 151.4 mm to (99.5, 107.8)
- moved L2 151.4 mm to (122.7, 84.0)
- moved L7 151.4 mm to (122.7, 116.0)
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Routing:
- net Net-(D10-Pin_1): track 5.11 -> 7.10 mm
- net VCC-: track 0.00 -> 0.92 mm, vias 0 -> 1
- net VCC+: track 0.00 -> 0.92 mm, vias 0 -> 1
- net GND: vias 343 -> 342
- added copper zone on B.Cu, net GND
Other:
- board text added: "Universal Machine Intelligence Dual DC LISN 9 kHz - 200 MHz ${REVISION}"
