File: lisn.kicad_sch (KiCad schematic)
At the start: 76 parts, among them X1 SMA, X10 Coax, X11 Coax, X12 Coax, X13 Contact, X14 Contact, X15 Contact, X16 Contact, X2 Conn_01x01, X3 Conn_01x01, X4 691313710002, X5 Conn_01x01, X6 Conn_01x01, X7 Conn_01x01, X8 Coax, X9 Coax

Commit message: finalize cleanup
Parts:
- added N1: 1590N1BK, symbol Mechanical:Housing
- added R50, R51: 470kR, Resistor_SMD:R_0603_1608Metric, symbol Device:R_Small_US
- C10, C6, C7, C9: Element14 (none) -> 4061686
- C11, C12, C3, C4: Element14 (none) -> 2812575; Mouser (none) -> 710-885342208004
- C5, C8: Element14 (none) -> 4061464
- D10, D11: Element14 (none) -> 3807475
- L1, L12: Element14 (none) -> 2894655
- L10, L11, L2, L3, L4, L5, L6, L7, L8, L9: Element14 (none) -> 2211603; Mouser (none) -> 710-744314110
- R1, R13: Element14 (none) -> 2303136
- R10, R22: Element14 (none) -> 2303090
- R11, R12, R23, R24: Element14 (none) -> 2059312
- R14, R2: Element14 (none) -> 2303084
- R15, R16, R3, R4: Element14 (none) -> 2303131
- R17, R5: Element14 (none) -> 2302967
- R18: Element14 (none) -> 4757417
- R19, R7: Element14 (none) -> 2302988
- R20, R8: Element14 (none) -> 2303141
- R21, R9: Element14 (none) -> 2303096
- R6: renamed from RR6; value 6 -> 27R; Element14 (none) -> 4757417
- X1: Element14 (none) -> 3583891
- X10, X11, X12, X9: footprint (none) -> Jumper_Coax:Jumper_RG178
- X13, X14, X15, X16: footprint TestPoint:TestPoint_Keystone_5019_Miniature -> SpringContact_Wurth:Wurth_331161702513; Element14 (none) -> 2249906
- X2: value Conn_01x01 -> 23.3000-22; footprint Connector:Banana_Jack_1Pin -> Connector_STAUBLI:STAUBLI_23.3000-22_Red; Element14 (none) -> 3223234
- X3: value Conn_01x01 -> 23.3000-22; footprint (none) -> Connector_STAUBLI:STAUBLI_23.3000-22_Red; Element14 (none) -> 3223234
- X4: Element14 (none) -> 1641993
- X5, X6: value Conn_01x01 -> 23.3000-21; footprint (none) -> Connector_STAUBLI:STAUBLI_23.3000-21_Black; Element14 (none) -> 3223233
- X7: value Conn_01x01 -> 23.3000-24; footprint (none) -> Connector_STAUBLI:STAUBLI_23.3000-24_Yellow; Element14 (none) -> 3276553
- X8: value Coax -> SMA; Element14 (none) -> 3583891
Connections:
- net GND: now also R50.2, R51.1
- net VCC+: now also R50.1
- net VCC-: now also R51.2
Other:
- note added: "RG 178 43mm"
- note added: "RG 178 52mm"
- company: (none) -> Universal Machine Intelligence
- title: (none) -> Dual DC LISN
- moved on the sheet: C1, C10, C11, C12, C13, C14, C2, C3, C4, C5, C6, C7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
